File: rfm69-rpi.sch (KiCad schematic (older format))
At the start: 21 parts, among them IC1 RFM69, IC2 RFM69, IC3 RFM69, IC4 RFM69, IC5 NCP1117, IC6 74HC139, J1 RPi_GPIO, P1 COAX, P2 COAX, P3 COAX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

Commit message: Version 2.0
Other:
- moved on the sheet: P5, R1, U1, U2
Changed lines of the file:
@@
 encoding utf-8
 Sheet 1 1
-Title "Raspberry Pi RFM69 Board"
+Title "Raspberry Pi RFM69 Interface"
 Date "2016-09-12"
 Rev "2.0"
@@
 $EndComp
 Wire Wire Line
-	6400 1550 6600 1550
+	6400 1550 6650 1550
 Wire Wire Line
 	6400 1950 6600 1950
@@
 Wire Wire Line
 	4500 1750 4300 1750
-Text GLabel 4500 2250 0    60   BiDi ~ 0
+Text GLabel 4500 2250 0    60   Output ~ 0
 MOSI
-Text GLabel 4500 2350 0    60   BiDi ~ 0
+Text GLabel 4500 2350 0    60   Input ~ 0
 MISO
 Text GLabel 4500 2450 0    60   Output ~ 0
 SCK
-Text GLabel 2600 1550 2    60   BiDi ~ 0
+Text GLabel 2600 1550 2    60   Input ~ 0
 MOSI
 Text GLabel 2600 1750 2    60   Input ~ 0
@@
 Wire Wire Line
 	2600 5550 3000 5550
-Text GLabel 2600 2750 2    60   BiDi ~ 0
+Text GLabel 2600 2750 2    60   Input ~ 0
 MOSI
-Text GLabel 2600 3950 2    60   BiDi ~ 0
+Text GLabel 2600 3950 2    60   Input ~ 0
 MOSI
-Text GLabel 2600 5150 2    60   BiDi ~ 0
+Text GLabel 2600 5150 2    60   Input ~ 0
 MOSI
-Text GLabel 2600 2850 2    60   BiDi ~ 0
+Text GLabel 2600 2850 2    60   Output ~ 0
 MISO
-Text GLabel 2600 4050 2    60   BiDi ~ 0
+Text GLabel 2600 4050 2    60   Output ~ 0
 MISO
-Text GLabel 2600 5250 2    60   BiDi ~ 0
+Text GLabel 2600 5250 2    60   Output ~ 0
 MISO
 Text GLabel 2600 2950 2    60   Input ~ 0
@@
 L Earth #PWR021
 U 1 1 57D5BD89
-P 8050 5800
-F 0 "#PWR021" H 8050 5550 50  0001 C CNN
-F 1 "Earth" H 8050 5650 50  0001 C CNN
-F 2 "" H 8050 5800 50  0000 C CNN
-F 3 "" H 8050 5800 50  0000 C CNN
-	1    8050 5800
+P 10400 5900
+F 0 "#PWR021" H 10400 5650 50  0001 C CNN
+F 1 "Earth" H 10400 5750 50  0001 C CNN
+F 2 "" H 10400 5900 50  0000 C CNN
+F 3 "" H 10400 5900 50  0000 C CNN
+	1    10400 5900
 	-1   0    0    1
 $EndComp
@@
 L CONN_01X02 P5
 U 1 1 57D5BC58
-P 8100 6000
-F 0 "P5" H 8100 6150 50  0000 C CNN
-F 1 "POWER" V 8200 6000 50  0000 C CNN
-F 2 "tinkerforge:JST-PH-SM4-2" H 8100 6000 50  0001 C CNN
-F 3 "" H 8100 6000 50  0000 C CNN
-	1    8100 6000
+P 10450 6100
+F 0 "P5" H 10450 6250 50  0000 C CNN
+F 1 "POWER" V 10550 6100 50  0000 C CNN
+F 2 "tinkerforge:JST-PH-SM4-2" H 10450 6100 50  0001 C CNN
+F 3 "" H 10450 6100 50  0000 C CNN
+	1    10450 6100
 	0    1    1    0
 $EndComp
@@
 NoConn ~ 8000 2250
 NoConn ~ 8000 2350
-Text GLabel 2600 1650 2    60   BiDi ~ 0
+Text GLabel 2600 1650 2    60   Output ~ 0
 MISO
 Connection ~ 4250 1150
@@
 L R R1
 U 1 1 57D5E166
-P 5400 5200
-F 0 "R1" V 5480 5200 50  0000 C CNN
-F 1 "4k7" V 5400 5200 50  0000 C CNN
-F 2 "agg:0805" V 5330 5200 50  0001 C CNN
-F 3 "" H 5400 5200 50  0000 C CNN
-	1    5400 5200
+P 5200 4450
+F 0 "R1" V 5280 4450 50  0000 C CNN
+F 1 "4k7" V 5200 4450 50  0000 C CNN
+F 2 "agg:0805" V 5130 4450 50  0001 C CNN
+F 3 "" H 5200 4450 50  0000 C CNN
+	1    5200 4450
 	1    0    0    -1
 $EndComp
@@
 L +3V3 #PWR027
 U 1 1 57D5E2C4
-P 5400 5050
-F 0 "#PWR027" H 5400 4900 50  0001 C CNN
-F 1 "+3V3" H 5400 5190 50  0000 C CNN
-F 2 "" H 5400 5050 50  0000 C CNN
-F 3 "" H 5400 5050 50  0000 C CNN
-	1    5400 5050
-	1    0    0    -1
-$EndComp
-Text GLabel 5300 5350 0    60   BiDi ~ 0
+P 5200 4300
+F 0 "#PWR027" H 5200 4150 50  0001 C CNN
+F 1 "+3V3" H 5200 4440 50  0000 C CNN
+F 2 "" H 5200 4300 50  0000 C CNN
+F 3 "" H 5200 4300 50  0000 C CNN
+	1    5200 4300
+	1    0    0    -1
+$EndComp
+Text GLabel 5100 4600 0    60   BiDi ~ 0
 ONEWIRE
 Wire Wire Line
-	5300 5350 5550 5350
+	5100 4600 5350 4600
 Connection ~ 6600 1550
 Connection ~ 2600 5450
@@
 L DS18B20 U1
 U 1 1 57D60AD9
-P 6000 5450
-F 0 "U1" H 5850 5700 50  0000 C CNN
-F 1 "1-Wire" H 6000 5200 50  0000 C CNN
-F 2 "TO_SOT_Packages_THT:TO-92_Molded_Narrow" H 5850 5700 50  0001 C CNN
-F 3 "" H 5850 5700 50  0000 C CNN
-	1    6000 5450
+P 5800 4700
+F 0 "U1" H 5650 4950 50  0000 C CNN
+F 1 "1-Wire" H 5800 4450 50  0000 C CNN
+F 2 "TO_SOT_Packages_THT:TO-92_Molded_Narrow" H 5650 4950 50  0001 C CNN
+F 3 "" H 5650 4950 50  0000 C CNN
+	1    5800 4700
 	1    0    0    -1
 $EndComp
@@
 L DS18B20 U2
 U 1 1 57D60D02
-P 6000 6100
-F 0 "U2" H 5850 6350 50  0000 C CNN
-F 1 "1-Wire" H 6000 5850 50  0000 C CNN
-F 2 "TO_SOT_Packages_THT:TO-92_Molded_Narrow" H 5850 6350 50  0001 C CNN
-F 3 "" H 5850 6350 50  0000 C CNN
-	1    6000 6100
-	1    0    0    -1
-$EndComp
-Wire Wire Line
-	5550 5350 5550 6100
-Wire Wire Line
-	5550 5450 5700 5450
-Connection ~ 5400 5350
-Wire Wire Line
-	5550 6100 5700 6100
-Connection ~ 5550 5450
+P 5800 5350
+F 0 "U2" H 5650 5600 50  0000 C CNN
+F 1 "1-Wire" H 5800 5100 50  0000 C CNN
+F 2 "TO_SOT_Packages_THT:TO-92_Molded_Narrow" H 5650 5600 50  0001 C CNN
+F 3 "" H 5650 5600 50  0000 C CNN
+	1    5800 5350
+	1    0    0    -1
+$EndComp
+Wire Wire Line
+	5350 4600 5350 5350
+Wire Wire Line
+	5350 4700 5500 4700
+Connection ~ 5200 4600
+Wire Wire Line
+	5350 5350 5500 5350
+Connection ~ 5350 4700
 $Comp
 L +3V3 #PWR032
 U 1 1 57D60DFF
-P 5700 5350
-F 0 "#PWR032" H 5700 5200 50  0001 C CNN
-F 1 "+3V3" H 5700 5490 50  0000 C CNN
-F 2 "" H 5700 5350 50  0000 C CNN
-F 3 "" H 5700 5350 50  0000 C CNN
-	1    5700 5350
+P 5500 4600
+F 0 "#PWR032" H 5500 4450 50  0001 C CNN
+F 1 "+3V3" H 5500 4740 50  0000 C CNN
+F 2 "" H 5500 4600 50  0000 C CNN
+F 3 "" H 5500 4600 50  0000 C CNN
+	1    5500 4600
 	1    0    0    -1
 $EndComp
@@
 L +3V3 #PWR033
 U 1 1 57D60E4C
-P 5700 6000
-F 0 "#PWR033" H 5700 5850 50  0001 C CNN
-F 1 "+3V3" H 5700 6140 50  0000 C CNN
-F 2 "" H 5700 6000 50  0000 C CNN
-F 3 "" H 5700 6000 50  0000 C CNN
-	1    5700 6000
+P 5500 5250
+F 0 "#PWR033" H 5500 5100 50  0001 C CNN
+F 1 "+3V3" H 5500 5390 50  0000 C CNN
+F 2 "" H 5500 5250 50  0000 C CNN
+F 3 "" H 5500 5250 50  0000 C CNN
+	1    5500 5250
 	1    0    0    -1
 $EndComp
@@
 L Earth #PWR034
 U 1 1 57D60EE1
-P 5700 6200
-F 0 "#PWR034" H 5700 5950 50  0001 C CNN
-F 1 "Earth" H 5700 6050 50  0001 C CNN
-F 2 "" H 5700 6200 50  0000 C CNN
-F 3 "" H 5700 6200 50  0000 C CNN
-	1    5700 6200
+P 5500 5450
+F 0 "#PWR034" H 5500 5200 50  0001 C CNN
+F 1 "Earth" H 5500 5300 50  0001 C CNN
+F 2 "" H 5500 5450 50  0000 C CNN
+F 3 "" H 5500 5450 50  0000 C CNN
+	1    5500 5450
 	1    0    0    -1
 $EndComp
@@
 L Earth #PWR035
 U 1 1 57D60F2E
-P 5700 5550
-F 0 "#PWR035" H 5700 5300 50  0001 C CNN
-F 1 "Earth" H 5700 5400 50  0001 C CNN
-F 2 "" H 5700 5550 50  0000 C CNN
-F 3 "" H 5700 5550 50  0000 C CNN
-	1    5700 5550
+P 5500 4800
+F 0 "#PWR035" H 5500 4550 50  0001 C CNN
+F 1 "Earth" H 5500 4650 50  0001 C CNN
+F 2 "" H 5500 4800 50  0000 C CNN
+F 3 "" H 5500 4800 50  0000 C CNN
+	1    5500 4800
 	1    0    0    -1
 $EndComp
@@
 L +5V #PWR036
 U 1 1 57D5BD4B
-P 8150 5800
-F 0 "#PWR036" H 8150 5650 50  0001 C CNN
-F 1 "+5V" H 8150 5940 50  0000 C CNN
-F 2 "" H 8150 5800 50  0000 C CNN
-F 3 "" H 8150 5800 50  0000 C CNN
-	1    8150 5800
+P 10500 5900
+F 0 "#PWR036" H 10500 5750 50  0001 C CNN
+F 1 "+5V" H 10500 6040 50  0000 C CNN
+F 2 "" H 10500 5900 50  0000 C CNN
+F 3 "" H 10500 5900 50  0000 C CNN
+	1    10500 5900
 	1    0    0    -1
 $EndComp
 Connection ~ 10450 5100
 Connection ~ 9450 5100
+$Comp
+L PWR_FLAG #FLG037
+U 1 1 57D7EA71
+P 6650 1550
+F 0 "#FLG037" H 6650 1645 50  0001 C CNN
+F 1 "PWR_FLAG" H 6650 1730 50  0000 C CNN
+F 2 "" H 6650 1550 50  0000 C CNN
+F 3 "" H 6650 1550 50  0000 C CNN
+	1    6650 1550
+	0    1    1    0
+$EndComp
+$Comp
+L PWR_FLAG #FLG038
+U 1 1 57D7ED23
+P 4500 1100
+F 0 "#FLG038" H 4500 1195 50  0001 C CNN
+F 1 "PWR_FLAG" H 4500 1280 50  0000 C CNN
+F 2 "" H 4500 1100 50  0000 C CNN
+F 3 "" H 4500 1100 50  0000 C CNN
+	1    4500 1100
+	1    0    0    -1
+$EndComp
+Wire Wire Line
+	4500 1100 4500 1350
+Connection ~ 4500 1350
 $EndSCHEMATC
